Commit message: feat(module2): develop Gazebo simulation content and examples
Develops the content and code examples for Module 2: The Digital Twin (Gazebo & Unity).

This includes:
- Content for Chapter 1 (Gazebo Basics) (T016).
- Content for Chapter 2 (Physics Simulation) (T017).
- Content for Chapter 3 (URDF and SDF Formats) and associated SDF example (T018).
- Content for Chapter 4 (Unity Visualization) (T019).
- Content for Chapter 5 (Sensor Simulation) and updated humanoid URDF with sensors (T020).
- Marks T016 to T020 as completed in tasks.md.

File: hackathone-ai-book/humanoid-robotics-book/static/code-examples/module1/ch5_urdf/generic_humanoid.urdf.xacro (robot description, xacro)
@@ -59,3 +59,163 @@
   </joint>
   <xacro:cylinder_link name="right_forearm_link" mass="${body_mass/6}" length="${body_len}" radius="${body_rad/4}"/>
+  <!-- Depth Camera Joint and Link -->
+  <joint name="camera_joint" type="fixed">
+    <parent link="head_link"/>
+    <child link="camera_link"/>
+    <origin xyz="0.05 0 0" rpy="0 0 0"/>
+  </joint>
+  <link name="camera_link">
+    <visual>
+      <geometry>
+        <box size="0.02 0.05 0.05"/>
+      </geometry>
+      <material name="red">
+        <color rgba="1 0 0 1"/>
+      </material>
+    </visual>
+  </link>
+  <!-- Gazebo Camera Sensor -->
+  <gazebo reference="camera_link">
+    <sensor name="depth_camera" type="depth">
+      <update_rate>30.0</update_rate>
+      <camera name="head_camera">
+        <horizontal_fov>1.047</horizontal_fov>
+        <image>
+          <width>640</width>
+          <height>480</height>
+          <format>R8G8B8</format>
+        </image>
+        <clip>
+          <near>0.1</near>
+          <far>10</far>
+        </clip>
+        <noise>
+          <type>gaussian</type>
+          <mean>0.0</mean>
+          <stddev>0.007</stddev>
+        </noise>
+      </camera>
+      <plugin name="camera_controller" filename="libgazebo_ros_camera.so">
+        <ros>
+          <namespace>camera</namespace>
+          <argument>--ros-args -r image:=image_raw -r depth_image:=depth/image_raw</argument>
+          <argument>--ros-args -r camera_info:=camera_info -r depth/camera_info:=depth/camera_info</argument>
+        </ros>
+        <camera_name>depth_camera</camera_name>
+        <frame_name>camera_depth_frame</frame_name>
+        <hack_baseline>0.07</hack_baseline>
+        <min_depth>0.1</min_depth>
+        <max_depth>10.0</max_depth>
+      </plugin>
+    </sensor>
+  </gazebo>
+  <!-- LiDAR Joint and Link -->
+  <joint name="laser_joint" type="fixed">
+    <parent link="torso_link"/>
+    <child link="laser_link"/>
+    <origin xyz="0.1 0 0.1" rpy="0 0 0"/>
+  </joint>
+  <link name="laser_link">
+    <visual>
+      <geometry>
+        <cylinder radius="0.03" length="0.04"/>
+      </geometry>
+      <material name="green">
+        <color rgba="0 1 0 1"/>
+      </material>
+    </visual>
+  </link>
+  <!-- Gazebo LiDAR Sensor -->
+  <gazebo reference="laser_link">
+    <sensor name="lidar" type="ray">
+      <pose>0 0 0 0 0 0</pose>
+      <visualize>true</visualize>
+      <update_rate>10.0</update_rate>
+      <ray>
+        <scan>
+          <horizontal>
+            <samples>640</samples>
+            <resolution>1</resolution>
+            <min_angle>-1.5708</min_angle>
+            <max_angle>1.5708</max_angle>
+          </horizontal>
+        </scan>
+        <range>
+          <min>0.1</min>
+          <max>10.0</max>
+          <resolution>0.01</resolution>
+        </range>
+        <noise>
+          <type>gaussian</type>
+          <mean>0.0</mean>
+          <stddev>0.01</stddev>
+        </noise>
+      </ray>
+      <plugin name="laser_controller" filename="libgazebo_ros_ray_sensor.so">
+        <ros>
+          <argument>--ros-args -r scan:=scan</argument>
+          <namespace>lidar</namespace>
+        </ros>
+        <output_type>sensor_msgs/LaserScan</output_type>
+        <frame_name>laser_frame</frame_name>
+      </plugin>
+    </sensor>
+  </gazebo>
+  <!-- Gazebo IMU Sensor (reference torso_link) -->
+  <gazebo reference="torso_link">
+    <sensor name="imu_sensor" type="imu">
+      <always_on>true</always_on>
+      <update_rate>100.0</update_rate>
+      <visualize>false</visualize>
+      <topic>imu</topic>
+      <plugin name="imu_plugin" filename="libgazebo_ros_imu_sensor.so">
+        <ros>
+          <namespace>/imu</namespace>
+          <argument>--ros-args -r imu:=data</argument>
+        </ros>
+        <frame_name>torso_link</frame_name>
+        <initial_orientation_as_reference>false</initial_orientation_as_reference>
+        <gyroscope>
+          <x>
+            <noise type="gaussian">
+              <mean>0.0</mean>
+              <stddev>0.0002</stddev>
+            </noise>
+          </x>
+          <y>
+            <noise type="gaussian">
+              <mean>0.0</mean>
+              <stddev>0.0002</stddev>
+            </noise>
+          </y>
+          <z>
+            <noise type="gaussian">
+              <mean>0.0</mean>
+              <stddev>0.0002</stddev>
+            </noise>
+          </z>
+        </gyroscope>
+        <accelerometer>
+          <x>
+            <noise type="gaussian">
+              <mean>0.0</mean>
+              <stddev>0.017</stddev>
+            </noise>
+          </x>
+          <y>
+            <noise type="gaussian">
+              <mean>0.0</mean>
+              <stddev>0.017</stddev>
+            </noise>
+          </y>
+          <z>
+            <noise type="gaussian">
+              <mean>0.0</mean>
+              <stddev>0.017</stddev>
+            </noise>
+          </z>
+        </accelerometer>
+      </plugin>
+    </sensor>
+  </gazebo>
 </robot>
